File: board/ME507-EMBER/ME507-EMBER.kicad_sch (KiCad schematic)
At the start: 20 parts, among them J1 Solenoid Terminal, J2 IR Cam Terminal, J3 External Power (12V), J4 DC Motor Terminal, J5 Encoder Terminal, Q2 Q_NMOS_SGD, U1 DRV8871DDA, U2 DRV8871DDA

Commit message: deleted:    board/ME507-EMBER/ME507-EMBER-backups/ME507-EMBER-2025-10-24_173205.zip 	new file:   board/ME507-EMBER/ME507-EMBER-backups/ME507-EMBER-2025-10-24_181717.zip 	new file:   board/ME507-EMBER/ME507-EMBER-backups/ME507-EMBER-2025-10-27_165905.zip 	new file:   board/ME507-EMBER/ME507-EMBER-backups/ME507-EMBER-2025-10-27_170905.zip 	new file:   board/ME507-EMBER/ME507-EMBER-backups/ME507-EMBER-2025-10-27_172403.zip 	new file:   board/ME507-EMBER/ME507-EMBER-backups/ME507-EMBER-2025-10-27_173500.zip 	new file:   board/ME507-EMBER/ME507-EMBER-backups/ME507-EMBER-2025-10-27_174108.zip 	modified:   board/ME507-EMBER/ME507-EMBER.kicad_pcb 	modified:   board/ME507-EMBER/ME507-EMBER.kicad_sch
Parts:
- added H1, H2, H3, H4: MountingHole, MountingHole:MountingHole_2.7mm_M2.5, symbol Mechanical:MountingHole
- added J6: IMU Terminal, TerminalBlock_Phoenix:TerminalBlock_Phoenix_MPT-0,5-4-2.54_1x04_P2.54mm_Horizontal, symbol Connector:Screw_Terminal_01x04
- added R5, R6: ~, Resistor_SMD:R_1206_3216Metric_Pad1.30x1.75mm_HandSolder, symbol Device:R_US
- J1: value Solenoid Terminal -> Solenoid
- U1, U2: value DRV8871DDA -> DRV8871
- renumbered ESP1 to ESP32, 4.7k4 to R1, 4.7k1 to R2, 4.7k2 to R3, 4.7k3 to R4, R1 to R7, R3 to R8, R2 to R9
Connections:
- net +3V3: now also J6.1 (Pin_1), R5.2, R6.2
- net GND: now also J6.2 (Pin_2)
- net at ESP32.33 (GPIO21/SDA), J2.3 (Pin_3): now also J6.3 (Pin_3), R5.1
- net at ESP32.36 (GPIO22/SCL), J2.4 (Pin_4): now also J6.4 (Pin_4), R6.1
Other:
- note added: "V_IMU (+) V_IMU (-) SDA SCL"

Commit message: new file:   board/ME507-EMBER/ME507-EMBER-backups/ME507-EMBER-2025-10-30_154305.zip 	new file:   board/ME507-EMBER/ME507-EMBER-backups/ME507-EMBER-2025-10-30_160009.zip 	new file:   board/ME507-EMBER/ME507-EMBER-backups/ME507-EMBER-2025-10-30_160613.zip 	new file:   board/ME507-EMBER/ME507-EMBER-backups/ME507-EMBER-2025-10-30_161352.zip 	new file:   board/ME507-EMBER/ME507-EMBER-backups/ME507-EMBER-2025-10-30_162427.zip 	modified:   board/ME507-EMBER/ME507-EMBER.kicad_pcb 	modified:   board/ME507-EMBER/ME507-EMBER.kicad_prl 	modified:   board/ME507-EMBER/ME507-EMBER.kicad_sch
Parts:
- removed Q2: Q_NMOS_SGD, EMBER_Footprints:MOSFET_Vishay_PowerPAK_1212-8_Single_JACKSON, symbol Transistor_FET:Q_NMOS_SGD
- added Q1: Q_NMOS_GDS, Package_TO_SOT_SMD:TO-252-2, symbol Transistor_FET:Q_NMOS_GDS
Connections:
- net GND: now also Q1.3 (S)
- net Q_D: now also Q1.2 (D)
- net at R7.2: now also Q1.1 (G)
Changed lines of the file:
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@@
-	)
-	(symbol
-		(lib_id "Transistor_FET:Q_NMOS_SGD")
-		(at 171.45 81.28 0)
-		(unit 1)
-		(exclude_from_sim no)
-		(in_bom yes)
-		(on_board yes)
-		(dnp no)
-		(fields_autoplaced yes)
-		(property "Reference" "Q2"
-			(at 177.8 80.0099 0)
-			(effects
-				(font
-					(size 1.27 1.27)
-				)
-				(justify left)
-			)
-		)
-		(property "Value" "Q_NMOS_SGD"
-			(at 177.8 82.5499 0)
-			(effects
-				(font
-					(size 1.27 1.27)
-				)
-				(justify left)
-			)
-		)
-		(property "Footprint" "EMBER_Footprints:MOSFET_Vishay_PowerPAK_1212-8_Single_JACKSON"
-			(at 176.53 78.74 0)
-			(effects
-				(font
-					(size 1.27 1.27)
-				)
-				(hide yes)
-			)
-		)
-		(property "Datasheet" "~"
-			(at 171.45 81.28 0)
-			(effects
-				(font
-					(size 1.27 1.27)
-				)
-				(hide yes)
-			)
-		)
-		(property "Description" "N-MOSFET transistor, source/gate/drain"
-			(at 171.45 81.28 0)
-			(effects
-				(font
-					(size 1.27 1.27)
-				)
-				(hide yes)
-			)
-		)
-		(pin "3"
-		)
-		(pin "1"
-		)
-		(pin "2"
-		)
-		(instances
-			(project ""
-				(path "/259d0011-820b-41ae-9d34-b870aa68bb26"
-					(reference "Q2")
-					(unit 1)
-				)
-			)
-		)
 	)
 	(symbol
@@
 					(unit 1)
 				)
+			)
+		)
+	)
+	(symbol
+		(lib_id "Transistor_FET:Q_NMOS_GDS")
+		(at 171.45 81.28 0)
+		(unit 1)
+		(exclude_from_sim no)
+		(in_bom yes)
+		(on_board yes)
+		(dnp no)
+		(fields_autoplaced yes)
+		(property "Reference" "Q1"
+			(at 177.8 80.0099 0)
+			(effects
+				(font
+					(size 1.27 1.27)
+				)
+				(justify left)
+			)
+		)
+		(property "Value" "Q_NMOS_GDS"
+			(at 177.8 82.5499 0)
+			(effects
+				(font
+					(size 1.27 1.27)
+				)
+				(justify left)
+			)
+		)
+		(property "Footprint" "Package_TO_SOT_SMD:TO-252-2"
+			(at 176.53 78.74 0)
+			(effects
+				(font
+					(size 1.27 1.27)
+				)
+				(hide yes)
+			)
+		)
+		(property "Datasheet" "~"
+			(at 171.45 81.28 0)
+			(effects
+				(font
+					(size 1.27 1.27)
+				)
+				(hide yes)
+			)
+		)
+		(property "Description" "N-MOSFET transistor, gate/drain/source"
+			(at 171.45 81.28 0)
+			(effects
+				(font
+					(size 1.27 1.27)
+				)
+				(hide yes)
+			)
+		)
+		(pin "1"
+		)
+		(pin "3"
+		)
+		(pin "2"
+		)
+		(instances
+			(project ""
+				(path "/259d0011-820b-41ae-9d34-b870aa68bb26"
+					(reference "Q1")
+					(unit 1)
+				)
